File: schematic/Modulator.kicad_sch (KiCad schematic)
At the start: 28 parts, among them J1 VIDEO IN, J2 VIDEO OUT, J4 MA05-2, U1 74590N, U10 TXS0108EPW, U11 TXS0108EPW, U12 TXS0108EPW, U2 IDT72125, U3 74590N, U4 7404N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

Commit message: First draft of PCB routing
Parts:
- added D1: D_Zener, Diode_THT:D_DO-41_SOD81_P7.62mm_Horizontal, symbol Device:D_Zener
- added D2: D, Diode_THT:D_DO-41_SOD81_P7.62mm_Horizontal, symbol Device:D
- added J3: 10164359-00011LF, 10164359_00011LF:AMPHENOL_10164359-00011LF, symbol 10164359-00011LF:10164359-00011LF
- added J5: PJ-002B, CUI_PJ-002B, symbol PJ-002B:PJ-002B
- added R1, R3: 5.1kR, Resistor_THT:R_Axial_DIN0207_L6.3mm_D2.5mm_P10.16mm_Horizontal, symbol Device:R
- J4: footprint Modulator:MA05-2 -> AD9834:AD9834
- U2: footprint Modulator:SO28L -> Package_DIP:DIP-28_W7.62mm_LongPads
Connections:
- net +5V: now also D1.1 (K), D2.1 (K), J3.A9 (VBUS_A), J3.B9 (VBUS_B), J5.1
- net D5_3V3: now also U9.38 (GPIO20); no longer U9.37 (GPIO26)
- net D6_3V3: now also U9.37 (GPIO26); no longer U9.38 (GPIO20)
- net GND: now also D1.2 (A), D2.2 (A), J3.A12 (GND_A), J3.B12 (GND_B), J3.SH1 (SHIELD), J3.SH2 (SHIELD__1), J3.SH3 (SHIELD__2), J3.SH4 (SHIELD__3), J5.2, J5.3, R1.2, R3.2
- new net: J3.B5 (CC2), R3.1
- new net: J3.A5 (CC1), R1.1
Other:
- note added: "Barrel Jack Power Input"
- note added: "USB-C Power Input"
- moved on the sheet: C10, C11, C12, C13, C14, C7, C8, C9, U1B, U2B, U3B, U4G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

Commit message: Make room for SMA connectors on DDS board
Parts:
- R2: footprint Modulator:0207_12 -> Resistor_THT:R_Axial_DIN0207_L6.3mm_D2.5mm_P10.16mm_Horizontal; symbol Modulator-eagle-import:R-US_0207/12 -> Device:R
- X2: footprint Modulator:DIL14S -> Oscillator:Oscillator_DIP-14; symbol Modulator-eagle-import:XO-14 -> Oscillator:CXO_DIP14
Other:
- moved on the sheet: C3

Commit message: Add decoupling capacitors to level shifters
Parts:
- added C1, C15, C16, C17, C2, C6: 100nF, Modulator:C050-025X075, symbol Modulator-eagle-import:C-US050-025X075
Connections:
- net +3V3: now also C16.1, C2.1, C6.1
- net +5V: now also C1.1, C15.1, C17.1
- net GND: now also C1.2, C15.2, C16.2, C17.2, C2.2, C6.2

Commit message: Change some decoupling capacitors, and usb-c resistors to SMT
Parts:
- C1, C15, C16, C17, C2, C6: footprint Modulator:C050-025X075 -> Capacitor_SMD:C_0805_2012Metric_Pad1.18x1.45mm_HandSolder
- R1, R3: footprint Resistor_THT:R_Axial_DIN0207_L6.3mm_D2.5mm_P10.16mm_Horizontal -> Resistor_SMD:R_0805_2012Metric_Pad1.20x1.40mm_HandSolder
- renumbered U12 to U11, U11 to U12
Changed lines of the file:
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@@
 			)
 		)
-		(property "Footprint" "Modulator:C050-025X075"
+		(property "Footprint" "Capacitor_SMD:C_0805_2012Metric_Pad1.18x1.45mm_HandSolder"
 			(at 212.09 91.44 0)
 			(effects
@@
 			)
 		)
-		(property "Footprint" "Modulator:C050-025X075"
+		(property "Footprint" "Capacitor_SMD:C_0805_2012Metric_Pad1.18x1.45mm_HandSolder"
 			(at 250.19 91.44 0)
 			(effects
@@
 			)
 		)
-		(property "Footprint" "Resistor_THT:R_Axial_DIN0207_L6.3mm_D2.5mm_P10.16mm_Horizontal"
+		(property "Footprint" "Resistor_SMD:R_0805_2012Metric_Pad1.20x1.40mm_HandSolder"
 			(at 56.642 254 90)
 			(effects
@@
 			)
 		)
-		(property "Footprint" "Resistor_THT:R_Axial_DIN0207_L6.3mm_D2.5mm_P10.16mm_Horizontal"
+		(property "Footprint" "Resistor_SMD:R_0805_2012Metric_Pad1.20x1.40mm_HandSolder"
 			(at 12.192 254 90)
 			(effects
@@
 			)
 		)
-		(property "Footprint" "Modulator:C050-025X075"
+		(property "Footprint" "Capacitor_SMD:C_0805_2012Metric_Pad1.18x1.45mm_HandSolder"
 			(at 181.61 90.17 0)
 			(effects
@@
 			)
 		)
-		(property "Footprint" "Modulator:C050-025X075"
+		(property "Footprint" "Capacitor_SMD:C_0805_2012Metric_Pad1.18x1.45mm_HandSolder"
 			(at 146.05 92.71 0)
 			(effects
@@
 			)
 		)
-		(property "Footprint" "Modulator:C050-025X075"
+		(property "Footprint" "Capacitor_SMD:C_0805_2012Metric_Pad1.18x1.45mm_HandSolder"
 			(at 167.64 90.17 0)
 			(effects
@@
 			)
 		)
-		(property "Footprint" "Modulator:C050-025X075"
+		(property "Footprint" "Capacitor_SMD:C_0805_2012Metric_Pad1.18x1.45mm_HandSolder"
 			(at 228.6 91.44 0)
 			(effects
@@
 		(dnp no)
 		(fields_autoplaced yes)
-		(property "Reference" "U11"
+		(property "Reference" "U12"
 			(at 200.3141 147.32 0)
 			(effects
@@
 			(project ""
 				(path "/32684964-aee7-4cbe-bac8-9927a2ba3460"
-					(reference "U11")
+					(reference "U12")
 					(unit 1)
 				)
@@
 		(on_board yes)
 		(dnp no)
-		(property "Reference" "U12"
+		(property "Reference" "U11"
 			(at 242.2241 147.32 0)
 			(effects
@@
 			(project ""
 				(path "/32684964-aee7-4cbe-bac8-9927a2ba3460"
-					(reference "U12")
+					(reference "U11")
 					(unit 1)
 				)

Commit message: Update capacitor footprints
Parts:
- C10, C11, C12, C13, C14, C3, C4, C5, C7, C8, C9: footprint Modulator:C050-025X075 -> Capacitor_THT:C_Disc_D4.7mm_W2.5mm_P5.00mm
Changed lines of the file:
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@@
 			)
 		)
-		(property "Footprint" "Modulator:C050-025X075"
+		(property "Footprint" "Capacitor_THT:C_Disc_D4.7mm_W2.5mm_P5.00mm"
 			(at 22.86 25.4 0)
 			(effects
@@
 			)
 		)
-		(property "Footprint" "Modulator:C050-025X075"
+		(property "Footprint" "Capacitor_THT:C_Disc_D4.7mm_W2.5mm_P5.00mm"
 			(at 288.29 125.73 0)
 			(effects
@@
 			)
 		)
-		(property "Footprint" "Modulator:C050-025X075"
+		(property "Footprint" "Capacitor_THT:C_Disc_D4.7mm_W2.5mm_P5.00mm"
 			(at 290.83 90.17 0)
 			(effects
@@
 			)
 		)
-		(property "Footprint" "Modulator:C050-025X075"
+		(property "Footprint" "Capacitor_THT:C_Disc_D4.7mm_W2.5mm_P5.00mm"
 			(at 53.34 25.4 0)
 			(effects
@@
 			)
 		)
-		(property "Footprint" "Modulator:C050-025X075"
+		(property "Footprint" "Capacitor_THT:C_Disc_D4.7mm_W2.5mm_P5.00mm"
 			(at 99.06 25.4 0)
 			(effects
@@
 			)
 		)
-		(property "Footprint" "Modulator:C050-025X075"
+		(property "Footprint" "Capacitor_THT:C_Disc_D4.7mm_W2.5mm_P5.00mm"
 			(at 68.58 25.4 0)
 			(effects
@@
 			)
 		)
-		(property "Footprint" "Modulator:C050-025X075"
+		(property "Footprint" "Capacitor_THT:C_Disc_D4.7mm_W2.5mm_P5.00mm"
 			(at 7.62 25.4 0)
 			(effects
@@
 			)
 		)
-		(property "Footprint" "Modulator:C050-025X075"
+		(property "Footprint" "Capacitor_THT:C_Disc_D4.7mm_W2.5mm_P5.00mm"
 			(at 114.3 25.4 0)
 			(effects
@@
 			)
 		)
-		(property "Footprint" "Modulator:C050-025X075"
+		(property "Footprint" "Capacitor_THT:C_Disc_D4.7mm_W2.5mm_P5.00mm"
 			(at 201.93 214.63 0)
 			(effects
@@
 			)
 		)
-		(property "Footprint" "Modulator:C050-025X075"
+		(property "Footprint" "Capacitor_THT:C_Disc_D4.7mm_W2.5mm_P5.00mm"
 			(at 38.1 25.4 0)
 			(effects
@@
 		(exclude_from_sim no)
 		(in_bom yes)
-		(on_board yes)
+		(on_board no)
 		(dnp no)
 		(fields_autoplaced yes)
@@
 			)
 		)
-		(property "Footprint" "Modulator:C050-025X075"
+		(property "Footprint" "Capacitor_THT:C_Disc_D4.7mm_W2.5mm_P5.00mm"
 			(at 83.82 25.4 0)
 			(effects
